File: test/pcb/Display/Display.kicad_sch (KiCad schematic)
At the start: 11 parts, among them J1 Conn_01x10, J2 Conn_01x02, J3 Conn_01x02, U1 UG-2864ASWPG01

Commit message: Version 0.4.0
Parts:
- renumbered C3 to C1, C3 to C2, R10 to R1, R10 to R2

Commit message: Use steps variable
Other:
- title: (none) -> Display Test
Changed lines of the file:
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@@
 	(generator_version "9.0")
 	(paper "A4")
+	(title_block
+		(title "Display Test")
+		(date "2026-02-27")
+		(rev "${VERSION}")
+	)
 	(rectangle
 		(start 119.38 86.36)

Commit message: Rename test/LedControl to test/LedControl-g431
Parts:
- U1: footprint local:Connector-Flat-24_P0.5mm -> local:Connector-Flat-24-0.5mm
Changed lines of the file:
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@@
 			)
 		)
-		(property "Footprint" "local:Connector-Flat-24_P0.5mm"
+		(property "Footprint" "local:Connector-Flat-24-0.5mm"
 			(at 53.34 82.55 0)
 			(effects
